File: Main_Board/Teensy.kicad_sch (KiCad schematic)
At the start: 0 parts

Commit message: connected vin global variable
Parts:
- added U2: DEV-15583, DEV-15583:MODULE_DEV-15583, symbol shared_symbols:DEV-15583
Connections:
- new net ADC1: U2.14
- new net ADC2: U2.15
- new net ADC3: U2.16
- new net GND: U2.G1, U2.G2, U2.G3
- new net UART_RX: U2.0
- new net UART_TX: U2.1
- new net VBUS_5V: U2.VIN
