File: EMG_filter/EMG_filter.kicad_pcb (KiCad board)
At the start: 2 copper layers, 43 x 19.5 mm, 22 parts, among them J1 Conn_01x03_Pin, J2 Conn_01x03_Pin, J3 Conn_01x04_Pin, U1 AD620, U2 MCP6022

Commit message: tag
reviewed and added signatures
Other:
- board text added: "Jax Kaz and Maanas were here :)"
Changed lines of the file:
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@@
 		(layer "Edge.Cuts")
+	)
+	(gr_text "Jax Kaz and\nMaanas were here\n:)"
+		(at 100.5 116 0)
+		(layer "F.SilkS")
+		(effects
+			(font
+				(size 0.5 0.5)
+				(thickness 0.1)
+			)
+			(justify left bottom)
+		)
 	)
 	(segment

Commit message: cleaned up repo
Other:
- board text added: "UW BMESOC"
Changed lines of the file:
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@@
 		(layer "Edge.Cuts")
 	)
-	(gr_text "Jax Kaz and\nMaanas were here\n:)"
-		(at 100.5 116 0)
+	(gr_text "UW BMESOC"
+		(at 91.5 117.5 0)
 		(layer "F.SilkS")
 		(effects
+			(font
+				(size 2 2)
+				(thickness 0.3)
+			)
+			(justify left bottom)
+		)
+	)
+	(gr_text "Jax Kaz and\nMaanas were here\n:)"
+		(at 100 107.5 270)
+		(layer "F.SilkS")
+		(effects
